File: DriveboardUSB/DriveboardUSB.kicad_pcb (KiCad board)
At the start: 2 copper layers, 250 x 120 mm, 69 parts, among them M542H_X_1 M542H_Header, M542H_Y_1 M542H_Header, M542H_Z_1 M542H_Header

Commit message: running traces
Parts:
- moved JP_PWR_STPR_to_AUXAIR_1 40.0 mm to (206.5, 105.0), turned to 270 degrees
- moved JP_GND_STPR_to_AUXAIR_1 38.2 mm to (243.5, 105.0), turned to 90 degrees
- moved D1 22.9 mm to (244.3, 110.0)
- moved D2 15.2 mm to (244.3, 124.0)
- moved JP_5V_ext_TO_laser_1 12.3 mm to (40.0, 46.5)
- moved JP_GND_ext_TO_laser_1 11.8 mm to (35.0, 46.5)
- moved R12 9.33 mm to (112.0, 125.5)
- moved R10 7.42 mm to (96.0, 125.5)
- moved R11 7.42 mm to (108.0, 125.5)
- moved R24 7.35 mm to (119.0, 112.5)
- moved C3 7.00 mm to (109.0, 118.0)
- moved OPTO_Z_1 7.00 mm to (102.0, 121.0)
- moved R1 6.48 mm to (36.0, 125.5)
- moved R9 5.57 mm to (92.0, 125.5)
- moved R2 4.69 mm to (40.0, 125.5)
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Routing:
- net 5V_ext: track 0.00 -> 112.9 mm
- net Net-(R24-Pad1): track 0.00 -> 93.3 mm
- net PWR_AIR: track 0.00 -> 85.3 mm
- net PWR_AUX: track 0.00 -> 83.5 mm
- net PD6: track 0.62 -> 74.2 mm
- net GND_ext: track 51.3 -> 0.00 mm, vias 5 -> 0
- net A_X: track 73.0 -> 23.1 mm, vias 1 -> 0
- net A'_X: track 58.8 -> 14.1 mm, vias 1 -> 0
- net B_X: track 64.4 -> 23.3 mm
- net A_Z: track 65.1 -> 24.1 mm
- net A_Y: track 63.2 -> 24.1 mm
- net TL_laser: track 0.00 -> 37.2 mm
- net A'_Z: track 50.8 -> 15.1 mm, vias 1 -> 0
- net A'_Y: track 49.4 -> 15.1 mm, vias 1 -> 0
- net 5V_laser: track 9.05 -> 43.2 mm
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- added copper zone on B.Cu, net 5V_ext
- added copper zone on B.Cu, net GND_STPR
- added copper zone on F.Cu, net GND_ext
- added copper zone on F.Cu, net PWR_STPR
- added copper zone on B.Cu, net SHILD
- removed copper zone on F.Cu, net 24V
- removed copper zone on F.Cu, net 5V_ext
- removed copper zone on B.Cu, net GND_24V
- removed copper zone on B.Cu, net GND_ext

Commit message: all traces, beautifying
Parts:
- moved R13 7.17 mm to (117.5, 114.0), turned to 180 degrees
- moved R24 2.93 mm to (117.5, 110.0), turned to 180 degrees
Routing:
- net A'_Y: track 15.1 -> 85.6 mm, vias 0 -> 1
- net A'_Z: track 15.1 -> 79.2 mm, vias 0 -> 1
- net A_X: track 23.1 -> 82.9 mm, vias 0 -> 1
- net A_Y: track 24.1 -> 83.9 mm, vias 0 -> 1
- net A_Z: track 24.1 -> 81.9 mm, vias 0 -> 1
- net B'_Z: track 36.1 -> 91.2 mm, vias 0 -> 1
- net B'_Y: track 35.9 -> 90.0 mm, vias 0 -> 1
- net B_Z: track 23.7 -> 77.5 mm, vias 0 -> 1
- net A'_X: track 14.1 -> 56.6 mm, vias 0 -> 1
- net GND_AUXAIR: track 0.00 -> 40.2 mm, vias 0 -> 2
- net B_Y: track 23.7 -> 62.8 mm, vias 0 -> 1
- net B_X: track 23.3 -> 59.8 mm, vias 0 -> 1
- net B'_X: track 35.5 -> 69.4 mm, vias 0 -> 1
- net PWR_AIR: track 85.3 -> 102.2 mm
- net PWR_AUX: track 83.5 -> 98.3 mm
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- added copper zone on B.Cu, net GND_AUXAIR
- added copper zone on F.Cu, net PWR_AUXAIR
- added copper zone on B.Cu, net SHILD_stpr
Other:
- net class Driver: clearance 0.3 -> 0.2; trace_width 0.8 -> 0.9

Commit message: DRC'd
Parts:
- moved R13 17.5 mm to (117.0, 96.5)
- moved R24 17.0 mm to (117.0, 93.0)
Routing:
- net GND: track 81.4 -> 40.7 mm, vias 8 -> 11
- net A_Z: track 81.9 -> 105.7 mm
- net Net-(R13-Pad1): track 80.2 -> 95.7 mm
- net Net-(R24-Pad1): track 84.0 -> 96.8 mm
- net A_Y: track 83.9 -> 75.2 mm
- net PD4: track 65.7 -> 57.9 mm
- net PD6: track 67.8 -> 60.2 mm
- net PB2: track 184.9 -> 188.4 mm
- net B'_Y: track 90.0 -> 87.0 mm
- net B_X: track 59.8 -> 62.7 mm
- net A'_X: track 56.6 -> 58.9 mm
- net B'_X: track 69.4 -> 71.5 mm
- net PB0: track 161.4 -> 163.4 mm
- net PD7: track 68.8 -> 70.5 mm
- net A_X: track 82.9 -> 84.1 mm
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
Commit message: generated gerber for v17.02
Routing:
- net WP_laser: track 30.4 -> 31.5 mm
Other:
- board text added: "(optional)"
- board text added: "Nortd Labs 2017"
- board text added: "STEPPER POWER"
- board text added: "VALVE POWER"
- board text removed: "24V"
- board text removed: "Nortd Labs 2016"

Commit message: generated gerber for v17.02 - with mount holes
Parts:
- added Mount_1: MountingHole_3.2mm_M3, Mounting_Holes:MountingHole_3.2mm_M3, F.Cu at (29.0, 125.0)
- added Mount_2: MountingHole_3.2mm_M3, Mounting_Holes:MountingHole_3.2mm_M3, F.Cu at (124.0, 125.0)
- added Mount_3: MountingHole_3.2mm_M3, Mounting_Holes:MountingHole_3.2mm_M3, F.Cu at (244.0, 125.0)
- added Mount_4: MountingHole_3.2mm_M3, Mounting_Holes:MountingHole_3.2mm_M3, F.Cu at (244.0, 49.0)
- added Mount_5: MountingHole_3.2mm_M3, Mounting_Holes:MountingHole_3.2mm_M3, F.Cu at (124.0, 49.0)
- added Mount_6: MountingHole_3.2mm_M3, Mounting_Holes:MountingHole_3.2mm_M3, F.Cu at (29.0, 49.0)
- moved D2 6.00 mm to (244.3, 118.0)
Routing:
- net PWR_AUX: track 99.1 -> 104.3 mm
- net GND_AUXAIR: track 40.2 -> 42.4 mm
- net PWR_AIR: track 101.4 -> 99.3 mm
- net 5V_ext: track 112.9 -> 114.9 mm
- net B_X: track 62.7 -> 64.1 mm
- net A'_X: track 58.9 -> 59.5 mm

Commit message: RFQ, take 2
Parts:
- removed Mount_1, Mount_2, Mount_3, Mount_4, Mount_5, Mount_6: MountingHole_3.2mm_M3, Mounting_Holes:MountingHole_3.2mm_M3
- added M1: MOUNT, Connect:1pin, F.Cu at (29.0, 125.0)
- added M2: MOUNT, Connect:1pin, F.Cu at (124.0, 125.0)
- added M3: MOUNT, Connect:1pin, F.Cu at (244.0, 125.0)
- added M4: MOUNT, Connect:1pin, F.Cu at (244.0, 49.0)
- added M5: MOUNT, Connect:1pin, F.Cu at (124.0, 49.0)
- added M6: MOUNT, Connect:1pin, F.Cu at (29.0, 49.0)
Connections:
- JACK_AIR_1 pad 9: SHILD_stpr -> SHILD
- JACK_AUX_1 pad 9: SHILD_stpr -> SHILD
- JACK_STEPPER_X_1 pad 9: SHILD_stpr -> SHILD
- JACK_STEPPER_Y_1 pad 9: SHILD_stpr -> SHILD
- JACK_STEPPER_Z_1 pad 9: SHILD_stpr -> SHILD
Routing:
- net SHILD: track 0.00 -> 130.7 mm
- net GND_laser: track 41.8 -> 42.5 mm
- removed copper zone on B.Cu, net SHILD_stpr
- removed copper zone on F.Cu, net SHILD_stpr
Other:
- board text added: "DriveboardUSB v17.03"
- board text removed: "DriveboardUSB v17.02"
